File: Kicad/PCB view/PCB0205.kicad_pcb (KiCad board)
At the start: 2 copper layers, 12 parts, among them J1 Soil Mositure Sen, U1 MOUDLE-SEEEDUINO-XIAO-ESP32C3, U3 MOUDLE-SEEEDUINO-XIAO-ESP32C3

Commit message: Saved local changes before pulling
Parts:
- moved R1 1.04 mm to (174.5, 70.5)
Routing:
- net +3.3V: track 112.4 -> 96.0 mm
- net Net-(Brd1-SDA): track 13.6 -> 7.70 mm, vias 3 -> 2
- net Net-(U1-PA8_A4_D4_SDA): track 6.10 -> 5.38 mm
Other:
- board outline added: 72 x 35 mm
Changed lines of the file:
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@@
 		(tags "capacitor handsolder")
 		(property "Reference" "C2"
-			(at 0 -1.68 360)
+			(at 0 -1.68 0)
 			(layer "F.SilkS")
 			(effects
@@
 		(tags "capacitor handsolder")
 		(property "Reference" "C4"
-			(at 0 -1.68 360)
+			(at 0 -1.68 0)
 			(layer "F.SilkS")
 			(effects
@@
 		)
 		(property "Value" "C"
-			(at 0 1.68 360)
+			(at 0 1.68 0)
 			(layer "F.Fab")
 			(hide yes)
@@
 		)
 		(fp_text user "${REFERENCE}"
-			(at 0 0 360)
+			(at 0 0 0)
 			(layer "F.Fab")
 			(effects
@@
 		)
 		(property "Value" "C"
-			(at 0 1.68 360)
+			(at 0 1.68 0)
 			(layer "F.Fab")
 			(effects
@@
 		)
 		(fp_text user "${REFERENCE}"
-			(at 0 0 360)
+			(at 0 0 0)
 			(layer "F.Fab")
 			(effects
@@
 	(footprint "Resistor_SMD:R_0815_2038Metric_Pad1.20x4.05mm_HandSolder"
 		(layer "F.Cu")
-		(at 174.175 69.5)
+		(at 174.475 70.5)
 		(descr "Resistor SMD 0815 (2038 Metric), square (rectangular) end terminal, IPC_7351 nominal with elongated pad for handsoldering. (Body size source: https://www.susumu.co.jp/common/pdf/n_catalog_partition07_en.pdf), generated with kicad-footprint-generator")
 		(tags "resistor handsolder")
 		(property "Reference" "R1"
-			(at 0 -2.98 360)
+			(at 0 -2.98 0)
 			(layer "F.SilkS")
 			(effects
@@
 		)
 		(property "Value" "R"
-			(at 0 2.98 360)
+			(at 0 2.98 0)
 			(layer "F.Fab")
 			(effects
@@
 		)
 		(fp_text user "${REFERENCE}"
-			(at 0 0 360)
+			(at 0 0 0)
 			(layer "F.Fab")
 			(effects
@@
 		(tags "resistor handsolder")
 		(property "Reference" "R2"
-			(at 0 -2.98 360)
+			(at 0 -2.98 0)
 			(layer "F.SilkS")
 			(effects
@@
 		)
 		(property "Value" "R"
-			(at 0 2.98 360)
+			(at 0 2.98 0)
 			(layer "F.Fab")
 			(effects
@@
 		)
 		(fp_text user "${REFERENCE}"
-			(at 0 0 360)
+			(at 0 0 0)
 			(layer "F.Fab")
 			(effects
@@
 		)
 		(fp_text user "${REFERENCE}"
-			(at 0 0 360)
+			(at 0 0 0)
 			(layer "F.Fab")
 			(effects
@@
 		(at 155.665 130)
 		(property "Reference" "U3"
-			(at 9.3345 -21.7805 360)
+			(at 9.3345 -21.7805 0)
 			(layer "F.SilkS")
 			(effects
@@
 		)
 		(property "Value" "MOUDLE-SEEEDUINO-XIAO-ESP32C3"
-			(at 8.89 -10.795 360)
+			(at 8.89 -10.795 0)
 			(layer "F.Fab")
 			(effects
@@
 		)
 		(property "Footprint" "xiao ESP32C3_PCB:MOUDLE14P-SMD-2.54-21X17.8MM"
-			(at 0 0 360)
+			(at 0 0 0)
 			(layer "F.Fab")
 			(hide yes)
@@
 		)
 		(property "Datasheet" ""
-			(at 0 0 360)
+			(at 0 0 0)
 			(layer "F.Fab")
 			(hide yes)
@@
 		)
 		(property "Description" ""
-			(at 0 0 360)
+			(at 0 0 0)
 			(layer "F.Fab")
 			(hide yes)
@@
 	)
 	(gr_line
-		(start 204.5 56)
-		(end 141 56)
+		(start 188.5 107.5)
+		(end 188.5 132)
 		(stroke
 			(width 0.2)
@@
 	)
 	(gr_line
-		(start 188.5 107.5)
+		(start 151.5 132)
 		(end 188.5 132)
 		(stroke
@@
 	)
 	(gr_line
-		(start 141 89.5)
-		(end 141 92)
+		(start 188.5 107.5)
+		(end 151.5 107.5)
 		(stroke
 			(width 0.2)
@@
 	)
 	(gr_line
-		(start 204.5 92)
-		(end 204.5 56)
+		(start 151.5 107.5)
+		(end 151.5 132)
 		(stroke
 			(width 0.2)
@@
 	)
 	(gr_line
-		(start 151.5 132)
-		(end 188.5 132)
+		(start 207.5 88)
+		(end 207.5 57)
 		(stroke
-			(width 0.2)
+			(width 0.05)
 			(type default)
 		)
-		(layer "F.Cu")
+		(layer "Edge.Cuts")
 	)
 	(gr_line
-		(start 141 56)
-		(end 141 58)
+		(start 207.5 89.5)
+		(end 207.5 92)
 		(stroke
-			(width 0.2)
+			(width 0.05)
 			(type default)
 		)
-		(layer "F.Cu")
+		(layer "Edge.Cuts")
 	)
 	(gr_line
-		(start 188.5 107.5)
-		(end 151.5 107.5)
+		(start 135.5 92)
+		(end 207.5 92)
 		(stroke
-			(width 0.2)
+			(width 0.05)
 			(type default)
 		)
-		(layer "F.Cu")
+		(layer "Edge.Cuts")
 	)
 	(gr_line
-		(start 151.5 107.5)
-		(end 151.5 132)
+		(start 135.5 89.5)
+		(end 135.5 92)
 		(stroke
-			(width 0.2)
+			(width 0.05)
 			(type default)
 		)
-		(layer "F.Cu")
+		(layer "Edge.Cuts")
 	)
 	(gr_line
-		(start 141 92)
-		(end 204.5 92)
+		(start 207.5 89.5)
+		(end 207.5 88)
 		(stroke
-			(width 0.2)
+			(width 0.05)
 			(type default)
 		)
-		(layer "F.Cu")
+		(layer "Edge.Cuts")
 	)
 	(gr_line
-		(start 141 57)
-		(end 141 89.5)
+		(start 207.5 57)
+		(end 135.5 57)
 		(stroke
-			(width 0.2)
+			(width 0.05)
 			(type default)
 		)
-		(layer "F.Cu")
+		(layer "Edge.Cuts")
+	)
+	(gr_line
+		(start 135.5 57)
+		(end 135.5 89.5)
+		(stroke
+			(width 0.05)
+			(type default)
+		)
+		(layer "Edge.Cuts")
 	)
 	(segment
@@
 	)
 	(segment
-		(start 188.525 89.45)
-		(end 190.675 91.6)
-		(width 0.2)
-		(layer "F.Cu")
-		(net 2)
-	)
-	(segment
 		(start 173.705 118)
 		(end 179.5 118)
@@
 	)
 	(segment
-		(start 190.675 91.6)
-		(end 204.1 91.6)
-		(width 0.2)
-		(layer "F.Cu")
-		(net 2)
-	)
-	(segment
 		(start 197.7125 83.0375)
 		(end 197.675 83)
@@
 	)
 	(segment
-		(start 167.275 77.5)
-		(end 170.675 77.5)
+		(start 173.45 70.5)
+		(end 170.475 73.475)
 		(width 0.2)
 		(layer "F.Cu")
@@
 	)
 	(segment
-		(start 173.15 69.5)
-		(end 171.175 69.5)
+		(start 167.275 77.5)
+		(end 170 77.5)
 		(width 0.2)
 		(layer "F.Cu")
@@
 	)
 	(segment
-		(start 171.175 69.5)
-		(end 170.675 70)
+		(start 170.43 73.52)
+		(end 170.475 73.475)
 		(width 0.2)
 		(layer "F.Cu")
 		(net 3)
 	)
-	(via
-		(at 170.675 77.5)
-		(size 0.6)
-		(drill 0.3)
-		(layers "F.Cu" "B.Cu")
+	(segment
+		(start 170 77.5)
+		(end 170.5 77)
+		(width 0.2)
+		(layer "F.Cu")
 		(net 3)
 	)
 	(via
-		(at 170.675 70)
+		(at 170.5 77)
 		(size 0.6)
 		(drill 0.3)
@@
 	)
 	(via
-		(at 170.675 70)
+		(at 170.475 73.475)
 		(size 0.6)
 		(drill 0.3)
@@
 	)
 	(segment
-		(start 170.675 77.5)
-		(end 170.675 70)
-		(width 0.2)
-		(layer "B.Cu")
-		(net 3)
-	)
-	(segment
 		(start 171.11 74.96)
 		(end 173.15 77)
@@
 	)
 	(segment
-		(start 179.12 73.42)
-		(end 179.675 73.42)
+		(start 175.5 70.5)
+		(end 178.42 73.42)
 		(width 0.2)
 		(layer "F.Cu")
@@
 	)
 	(segment
-		(start 175.2 69.5)
-		(end 179.12 73.42)
+		(start 178.42 73.42)
+		(end 179.675 73.42)
 		(width 0.2)
 		(layer "F.Cu")

Commit message: Update Soil monitor project files
Parts:
- removed Brd1: SSD1306, SSD1306:128x64OLED
- removed C2, C4: C, Capacitor_SMD:C_0805_2012Metric_Pad1.18x1.45mm_HandSolder
- removed U3: MOUDLE-SEEEDUINO-XIAO-ESP32C3, xiao ESP32C3_PCB:MOUDLE14P-SMD-2.54-21X17.8MM
- added Brd2: SSD1306, SSD1306:128x64OLED, F.Cu at (98.1, 58.0)
- added SW1: SW_Push, Connector_PinHeader_2.54mm:PinHeader_1x03_P2.54mm_Vertical, F.Cu at (84.0, 75.5)
- added SW3: SW_SPDT, Connector_PinHeader_2.54mm:PinHeader_1x03_P2.54mm_Vertical, F.Cu at (172.7, 42.8)
- added U2: ~, 514_KiCAD_Demo:XIAO_ESP32_SENSE, F.Cu at (157.3, 66.8)
- D1: value WS2812B -> LED; footprint LED_SMD:LED_WS2812B_PLCC4_5.0x5.0mm_P3.2mm -> LED_SMD:LED_0805_2012Metric_Pad1.15x1.40mm_HandSolder
- J1: footprint Connector_PinHeader_2.54mm:PinHeader_1x03_P2.54mm_Vertical_SMD_Pin1Right -> Connector_PinHeader_2.54mm:PinHeader_1x03_P2.54mm_Vertical
- R1, R2, R3: footprint Resistor_SMD:R_0815_2038Metric_Pad1.20x4.05mm_HandSolder -> Resistor_SMD:R_0805_2012Metric_Pad1.20x1.40mm_HandSolder
- U1: value MOUDLE-SEEEDUINO-XIAO-ESP32C3 -> ~; footprint xiao ESP32C3_PCB:MOUDLE14P-SMD-2.54-21X17.8MM -> 514_KiCAD_Demo:XIAO_ESP32_SENSE
- moved D1 130.3 mm to (60.0, 81.0), turned to 180 degrees
- moved U1 114.0 mm to (65.6, 68.5)
- moved R2 107.2 mm to (67.0, 81.0), turned to 180 degrees
- moved R3 103.6 mm to (78.5, 75.0), turned to 90 degrees
- moved C3 88.2 mm to (83.5, 59.0), turned to 180 degrees
- moved J1 45.4 mm to (181.2, 65.4), turned to 180 degrees
- moved R1 29.7 mm to (154.7, 48.3)
- moved C1 27.3 mm to (175.7, 62.9), turned to -90 degrees
Connections:
- C1 pad 1: +3.3V -> GND
- C1 pad 2: GND -> +3.3V
- D1 pad 1: +3.3V -> Net-(D1-K)
- D1 pad 2: unconnected-(D1-DOUT-Pad2) -> Net-(D1-A)
- R1 pad 2: Net-(U1-PA8_A4_D4_SDA) -> +3.3V
- R2 pad 1: Net-(Brd1-SCL) -> GND
- R2 pad 2: Net-(U1-PA9_A5_D5_SCL) -> Net-(D1-K)
- R3 pad 1: Net-(U1-PB08_A6_D6_TX) -> Net-(U1-GPIO44_D7_RX)
- R3 pad 2: Net-(D1-DIN) -> +3.3V
- U1 pad 1: Net-(U1-PA02_A0_D0) -> unconnected-(U1-GPIO1_A0_D0-Pad1)
- U1 pad 10: unconnected-(U1-PA5_A9_D9_MISO-Pad10) -> +3.3V
- U1 pad 12: +3.3V -> unconnected-(U1-GPIO8_A9_D9_CIPO-Pad12)
- U1 pad 13: Net-(U1-GND) -> unconnected-(U1-GPIO7_A8_D8_SCK-Pad13)
- U1 pad 14: unconnected-(U1-5V-Pad14) -> Net-(U1-GPIO44_D7_RX)
- U1 pad 2: Net-(U1-PA4_A1_D1) -> unconnected-(U1-GPIO2_A1_D1-Pad2)
- U1 pad 3: Net-(U1-PA10_A2_D2) -> unconnected-(U1-GPIO3_A2_D2-Pad3)
- U1 pad 4: Net-(U1-PA11_A3_D3) -> unconnected-(U1-GPIO4_A3_D3-Pad4)
- U1 pad 5: Net-(U1-PA8_A4_D4_SDA) -> Net-(Brd2-SDA)
- U1 pad 6: Net-(U1-PA9_A5_D5_SCL) -> Net-(Brd2-SCL)
- U1 pad 7: Net-(U1-PB08_A6_D6_TX) -> Net-(D1-A)
- U1 pad 8: Net-(U1-PB09_A7_D7_RX) -> unconnected-(U1-5V-Pad8)
- U1 pad 9: unconnected-(U1-PA7_A8_D8_SCK-Pad9) -> GND
Routing:
- net Net-(Brd2-SDA): track 0.00 -> 51.0 mm
- net Net-(Brd2-SCL): track 0.00 -> 46.1 mm
- net GND: track 84.5 -> 38.8 mm, vias 5 -> 2
- net Net-(SW3-B): track 7.70 -> 34.3 mm, vias 2 -> 0
- net +3.3V: track 96.0 -> 78.8 mm
- net Net-(U1-GPIO44_D7_RX): track 0.00 -> 11.0 mm
- net /signal: track 32.7 -> 43.3 mm, vias 2 -> 0
- net Net-(D1-DIN): track 7.25 -> 0.00 mm
- net Net-(Brd1-SCL): track 6.72 -> 0.00 mm
- net Net-(D1-A): track 0.00 -> 5.88 mm
- net Net-(U1-PB08_A6_D6_TX): track 5.80 -> 0.00 mm
- net Net-(U1-PA8_A4_D4_SDA): track 5.38 -> 0.00 mm
- net Net-(D1-K): track 0.00 -> 4.95 mm
- net Net-(U1-PA9_A5_D5_SCL): track 4.91 -> 0.00 mm
- added copper zone on B.Cu, net GND
Other:
- board size 72 x 35 mm -> 63.5 x 39.5 mm
